File: ya4b/data-register/data-register-bank/data-register-bank.sch (KiCad schematic (older format))
At the start: 57 parts, among them J1 Conn_01x38, U1 GAL16V8, U10 74LS173, U2 GAL16V8, U3 74LS243, U4 74LS173, U5 74LS243, U6 74LS173, U7 74LS243, U8 74LS173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

Commit message: Updated schematic and pcb for data register bank; data pins were off by one
Connections:
- net Data0: now also J1.27 (Pin_27); no longer J1.26 (Pin_26)
- net Data1: now also J1.28 (Pin_28); no longer J1.27 (Pin_27)
- net Data2: now also J1.29 (Pin_29); no longer J1.28 (Pin_28)
- net Data3: now also J1.30 (Pin_30); no longer J1.29 (Pin_29)
Changed lines of the file:
@@
 Wire Wire Line
 	6250 8250 6250 8450
-NoConn ~ 6750 8450
 NoConn ~ 6850 8450
 NoConn ~ 6950 8450
@@
 	3350 1850 3600 1850
 Entry Wire Line
+	6750 8000 6850 7900
+Entry Wire Line
 	6650 8000 6750 7900
 Entry Wire Line
@@
 Entry Wire Line
 	6450 8000 6550 7900
-Entry Wire Line
-	6350 8000 6450 7900
-Wire Wire Line
-	6350 8000 6350 8450
 Wire Wire Line
 	6450 8000 6450 8450
@@
 Wire Wire Line
 	6650 8000 6650 8450
-Text Label 6350 8300 3    39   ~ 0
+Wire Wire Line
+	6750 8000 6750 8450
+Text Label 6450 8300 3    39   ~ 0
 Data0
-Text Label 6450 8300 3    39   ~ 0
+Text Label 6550 8300 3    39   ~ 0
 Data1
-Text Label 6550 8300 3    39   ~ 0
+Text Label 6650 8300 3    39   ~ 0
 Data2
-Text Label 6650 8300 3    39   ~ 0
+Text Label 6750 8300 3    39   ~ 0
 Data3
 Wire Bus Line
@@
 Wire Wire Line
 	5150 7650 4700 7650
-Wire Bus Line
-	6450 7900 8800 7900
+Connection ~ 4700 7650
+Connection ~ 8800 7900
+Wire Bus Line
+	8800 7900 8900 7900
+NoConn ~ 6350 8450
+Wire Bus Line
+	6550 7900 8800 7900
 Wire Bus Line
 	3250 1550 3250 5600
@@
 Wire Bus Line
 	5100 1550 5100 5600
-Connection ~ 4700 7650
 $EndSCHEMATC
