File: ya4b/data-register/data-register-bank/data-register-bank.kicad_pcb (KiCad board)
At the start: 4 copper layers, 99.6 x 59.1 mm, 57 parts, among them J1 Conn_01x38, U1 GAL16V8, U10 74LS173, U2 GAL16V8, U3 74LS243, U4 74LS173, U5 74LS243, U6 74LS173, U7 74LS243, U8 74LS173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

Commit message: Updated schematic and pcb for data register bank; data pins were off by one
Connections:
- J1 pad 26: /Data0 -> Net-(J1-Pad26)
- J1 pad 27: /Data1 -> /Data0
- J1 pad 28: /Data2 -> /Data1
- J1 pad 29: /Data3 -> /Data2
- J1 pad 30: Net-(J1-Pad30) -> /Data3
Routing:
- net /Data0: track 182.8 -> 185.4 mm
- net /Data1: track 182.3 -> 184.8 mm
- net /Data3: track 186.4 -> 188.9 mm
- net /Data2: track 183.5 -> 186.0 mm
Other:
- board text added: "YA4B Data Register Bank v1.0.1 © 2020 Gregory Martin"
- board text removed: "YA4B Data Register Bank v1.0 © 2020 Gregory Martin"

Commit message: Made a patched version of the data register bank output control GAL because of an error on the PCB design.
Created a design for the ALU in Digital that seems to work.
Other:
- board text added: "YA4B Data Register Bank v1.0.2 © 2020 Gregory Martin"
- board text removed: "YA4B Data Register Bank v1.0.1 © 2020 Gregory Martin"
Changed lines of the file:
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@@
     )
   )
-  (gr_text "YA4B Data Register Bank v1.0.1\n© 2020 Gregory Martin" (at 82.0801 179.7177) (layer F.SilkS)
+  (gr_text "YA4B Data Register Bank v1.0.2\n© 2020 Gregory Martin" (at 82.0801 179.7177) (layer F.SilkS)
     (effects (font (size 0.8 0.8) (thickness 0.15)))
   )
@@
   (gr_line (start 149.1234 187.3504) (end 149.1234 128.2954) (layer Edge.Cuts) (width 0.05))
   (gr_line (start 49.6316 187.325) (end 149.1234 187.3504) (layer Edge.Cuts) (width 0.05))
-  (gr_text D3 (at 123.7107 181.8386 90) (layer F.SilkS)
+  (gr_text D3 (at 126.0348 181.9783 90) (layer F.SilkS)
     (effects (font (size 1 1) (thickness 0.15)) (justify left))
   )
-  (gr_text D2 (at 121.2088 181.8386 90) (layer F.SilkS)
+  (gr_text D2 (at 123.5329 181.9783 90) (layer F.SilkS)
     (effects (font (size 1 1) (thickness 0.15)) (justify left))
   )
-  (gr_text D1 (at 118.6688 181.8386 90) (layer F.SilkS)
+  (gr_text D1 (at 121.031 181.9783 90) (layer F.SilkS)
     (effects (font (size 1 1) (thickness 0.15)) (justify left))
   )
-  (gr_text D0 (at 116.1161 181.8386 90) (layer F.SilkS)
+  (gr_text D0 (at 118.4656 181.9783 90) (layer F.SilkS)
     (effects (font (size 1 1) (thickness 0.15)) (justify left))
   )
